Commit message: changed collision geometry and Gazebo materials

File: src/skid4wd_description/urdf/materials.xacro (robot description, xacro)
@@ -1,6 +1,10 @@
 <?xml version="1.0" ?>
 <robot name="skid4wd" xmlns:xacro="http://www.ros.org/wiki/xacro" >
-<material name="silver">
-  <color rgba="0.700 0.700 0.700 1.000"/>
-</material>
+  <xacro:macro name="materials" params="name rgba">
+    <material name="${name}">
+      <color rgba="${rgba}"/>
+    </material>
+  </xacro:macro>
+<xacro:materials name="silver" rgba="0.700 0.700 0.700 1.000"/>
+<xacro:materials name="orange" rgba="1.0 0.423529411765 0.0392156862745 1.0"/>
 </robot>

File: src/skid4wd_description/urdf/skid4wd.xacro (robot description, xacro)
@@ -4,4 +4,5 @@
 <xacro:include filename="$(find skid4wd_description)/urdf/skid4wd.trans" />
 <xacro:include filename="$(find skid4wd_description)/urdf/skid4wd.gazebo" />
+<xacro:property name="PI" value="3.14"/>
 <link name="base_link">
   <inertial>
@@ -15,5 +16,5 @@
       <mesh filename="package://skid4wd_description/meshes/base_link.stl" scale="0.001 0.001 0.001"/>
     </geometry>
-    <material name="silver"/>
+    <material name="orange"/>
   </visual>
   <collision>
@@ -38,7 +39,7 @@
   </visual>
   <collision>
-    <origin rpy="0 0 0" xyz="-0.125 -0.16 -0.03"/>
+    <origin rpy="${PI/2} 0 0" xyz="0 0 0"/>
     <geometry>
-      <mesh filename="package://skid4wd_description/meshes/wheel_front_left_1.stl" scale="0.001 0.001 0.001"/>
+      <cylinder length="0.07" radius="0.08"/>
     </geometry>
   </collision>
@@ -58,7 +59,7 @@
   </visual>
   <collision>
-    <origin rpy="0 0 0" xyz="-0.125 0.16 -0.03"/>
+    <origin rpy="${PI/2} 0 0" xyz="0 0 0"/>
     <geometry>
-      <mesh filename="package://skid4wd_description/meshes/wheel_front_right_1.stl" scale="0.001 0.001 0.001"/>
+      <cylinder length="0.07" radius="0.08"/>
     </geometry>
   </collision>
@@ -78,7 +79,7 @@
   </visual>
   <collision>
-    <origin rpy="0 0 0" xyz="0.125 -0.16 -0.03"/>
+    <origin rpy="${PI/2} 0 0" xyz="0 0 0"/>
     <geometry>
-      <mesh filename="package://skid4wd_description/meshes/wheel_rear_left_1.stl" scale="0.001 0.001 0.001"/>
+      <cylinder length="0.07" radius="0.08"/>
     </geometry>
   </collision>
@@ -98,7 +99,7 @@
   </visual>
   <collision>
-    <origin rpy="0 0 0" xyz="0.125 0.16 -0.03"/>
+    <origin rpy="${PI/2} 0 0" xyz="0 0 0"/>
     <geometry>
-      <mesh filename="package://skid4wd_description/meshes/wheel_rear_right_1.stl" scale="0.001 0.001 0.001"/>
+      <cylinder length="0.07" radius="0.08"/>
     </geometry>
   </collision>
