Commit message: changed mesh file for wheel and added world config

File: src/skid4wd_description/urdf/skid4wd.xacro (robot description, xacro)
@@ -32,7 +32,7 @@
   </inertial>
   <visual>
-    <origin rpy="0 0 0" xyz="-0.125 -0.16 -0.03"/>
+    <origin rpy="0 0 0" xyz="-0.01 0.005 -0.017"/>
     <geometry>
-      <mesh filename="package://skid4wd_description/meshes/wheel_front_left_1.stl" scale="0.001 0.001 0.001"/>
+      <mesh filename="package://skid4wd_description/meshes/wheel.dae"/>
     </geometry>
     <material name="silver"/>
@@ -52,7 +52,7 @@
   </inertial>
   <visual>
-    <origin rpy="0 0 0" xyz="-0.125 0.16 -0.03"/>
+    <origin rpy="0 0 ${PI}" xyz="0.01 -0.005 -0.017"/>
     <geometry>
-      <mesh filename="package://skid4wd_description/meshes/wheel_front_right_1.stl" scale="0.001 0.001 0.001"/>
+      <mesh filename="package://skid4wd_description/meshes/wheel.dae"/>
     </geometry>
     <material name="silver"/>
@@ -72,7 +72,7 @@
   </inertial>
   <visual>
-    <origin rpy="0 0 0" xyz="0.125 -0.16 -0.03"/>
+    <origin rpy="0 0 0" xyz="-0.01 0.005 -0.017"/>
     <geometry>
-      <mesh filename="package://skid4wd_description/meshes/wheel_rear_left_1.stl" scale="0.001 0.001 0.001"/>
+      <mesh filename="package://skid4wd_description/meshes/wheel.dae"/>
     </geometry>
     <material name="silver"/>
@@ -92,7 +92,7 @@
   </inertial>
   <visual>
-    <origin rpy="0 0 0" xyz="0.125 0.16 -0.03"/>
+    <origin rpy="0 0 ${PI}" xyz="0.01 -0.005 -0.017"/>
     <geometry>
-      <mesh filename="package://skid4wd_description/meshes/wheel_rear_right_1.stl" scale="0.001 0.001 0.001"/>
+      <mesh filename="package://skid4wd_description/meshes/wheel.dae"/>
     </geometry>
     <material name="silver"/>

Commit message: added controller to robot

File: src/skid4wd_description/urdf/skid4wd.xacro (robot description, xacro)
@@ -110,4 +110,6 @@
   <child link="wheel_front_left_1"/>
   <axis xyz="0.0 1.0 0.0"/>
+  <limit effort="10000" velocity="1000"/>
+  <joint_properties damping="1.0" friction="1.0"/>
 </joint>
 <joint name="joint_front_right" type="continuous">
@@ -115,5 +117,7 @@
   <parent link="base_link"/>
   <child link="wheel_front_right_1"/>
-  <axis xyz="0.0 -1.0 0.0"/>
+  <axis xyz="0.0 1.0 0.0"/>
+  <limit effort="10000" velocity="1000"/>
+  <joint_properties damping="1.0" friction="1.0"/>
 </joint>
 <joint name="joint_rear_left" type="continuous">
@@ -122,4 +126,6 @@
   <child link="wheel_rear_left_1"/>
   <axis xyz="0.0 1.0 0.0"/>
+  <limit effort="10000" velocity="1000"/>
+  <joint_properties damping="1.0" friction="1.0"/>
 </joint>
 <joint name="joint_rear_right" type="continuous">
@@ -127,5 +133,7 @@
   <parent link="base_link"/>
   <child link="wheel_rear_right_1"/>
-  <axis xyz="0.0 -1.0 0.0"/>
+  <axis xyz="0.0 1.0 0.0"/>
+  <limit effort="10000" velocity="1000"/>
+  <joint_properties damping="1.0" friction="1.0"/>
 </joint>
 </robot>

Commit message: Add files via upload
added imu and depth camera

File: src/skid4wd_description/urdf/skid4wd.xacro (robot description, xacro)
@@ -137,3 +137,23 @@
   <joint_properties damping="1.0" friction="1.0"/>
 </joint>
+<!--  -->
+<joint name="camera_joint" type="fixed">
+    <parent link="base_link"/>
+    <child link="camera_link"/>
+    <origin xyz="0.305 0 0.08" rpy="0 0 0"/>
+</joint>
+<link name="camera_link">
+    <visual>
+        <geometry>
+            <box size="0.010 0.03 0.03"/>
+        </geometry>
+    </visual>
+</link>
+<joint name="camera_optical_joint" type="fixed">
+    <parent link="camera_link"/>
+    <child link="camera_link_optical"/>
+    <origin xyz="0 0 0" rpy="${-pi/2} 0 ${-pi/2}"/>
+</joint>
+<link name="camera_link_optical"></link>
+<!--  -->
 </robot>
